File: TEJ4M-Unit-4-07/TEJ4M-Unit-4-07-Backup.kicad_sch (KiCad schematic)
At the start: 14 parts, among them U1 4001, U2 4001, U3 ADG417BN, U4 ADG417BN

Commit message: Add files via upload
Parts:
- removed H1, H2, H3, H4: MountingHole_Pad, MountingHole:MountingHole_2.7mm_Pad, symbol Mechanical:MountingHole_Pad
- D1, D2: footprint LED_THT:LED_D1.8mm_W1.8mm_H2.4mm_Horizontal_O1.27mm_Z1.6mm -> (none)
- R1, R2, R3, R4: footprint Resistor_THT:R_Axial_DIN0204_L3.6mm_D1.6mm_P5.08mm_Horizontal -> (none)
- U1, U2: footprint Package_DIP:DIP-14_W10.16mm -> (none)
Connections:
- net +5V: now also R3.1, R4.1; no longer U3.1, U4.1
- net GND: no longer R3.1, R4.2
- net at U2.2, U4.8: no longer R3.2
- net at U1.1, U3.8: no longer R4.1
- new net: R3.2, U4.1
- new net: R4.2, U3.1
Other:
- moved on the sheet: R4, U3A, U4A
